File: hardware/PCB/Plug_Pass_120V_arduino_shield.kicad_pcb (KiCad board)
At the start: 2 copper layers, 134.6 x 108 mm, 8 parts, among them J1 Conn_01x06, J10 TDPT-1017503, J2 Conn_01x08, J3 Conn_02x04_Odd_Even, J4 Conn_02x04_Odd_Even

Commit message: KiCAD files from first prototype batch
Parts:
- removed J10: TDPT-1017503, Plug_Pass:TDPT_2P_5.08MM
- removed J4: Conn_02x04_Odd_Even, Plug_Pass:IDC-Header_2x04_P2.54mm_Vertical
- removed PS1: IRM-05-5, Plug_Pass:Converter_ACDC_MeanWell_IRM-05-xx_THT
- removed RLY1: T95S5D22-5, Plug_Pass:RLY-T9AS5D22-5
Routing:
- net Net-(J10-Pad1): track 42.1 -> 0.00 mm
- net VCC: track 60.9 -> 22.6 mm
- net Net-(J9-Pad~): track 35.8 -> 0.00 mm
- net /RelayPin: track 53.7 -> 20.1 mm
- net GNDREF: track 8.70 -> 0.00 mm
Other:
- board size 134.6 x 108 mm -> 40.6 x 108 mm
- board text added: "Plug Pass version 1.0 arduino shield"
