File: hardware/PCB/Plug_Pass.sch (KiCad schematic (older format))
At the start: 12 parts, among them J1 Conn_01x06, J10 TDPT-1017503, J2 Conn_01x08, J3 Conn_02x04_Odd_Even, J4 Conn_02x04_Odd_Even, J5 Conn_WallSocket_Earth, J8 QuickDisconnect, J9 QuickDisconnect

Commit message: Add files via upload
Parts:
- removed J10: TDPT-1017503, Plug_Pass:TDPT_2P_6.35MM, symbol Plug_Pass:TDPT-1017503
- added H1, H2, H3, H4: MountingHole_Pad, Plug_Pass:Ground_Pad, symbol Plug_Pass:MountingHole_Pad
- added J6: Screw_Terminal_01x01, Plug_Pass:PLH5-1_75, symbol Plug_Pass:Screw_Terminal_01x01
- A1: value Arduino_Nano_v3.x -> Arduino_Nano_Every; footprint Plug_Pass:Arduino_Nano_WithMountingHoles -> Plug_Pass:NANO_33_Footprint_SMD_Castell
- J1: footprint Plug_Pass:PinSocket_1x06_P2.54mm_Vertical -> Plug_Pass:RTC_PinHeader
- J2: footprint Plug_Pass:PinSocket_1x08_P2.54mm_Vertical -> Plug_Pass:PN532_NFC_PinSocket
- J3: footprint Plug_Pass:IDC-Header_2x04_P2.54mm_Vertical -> Plug_Pass:IDC-Header_2x04_P2.54mm_Vertical_Small
Connections:
- net Earth is gone; now on net GNDREF: J5.3 (EARTH)
- net GNDREF: now also J3.2 (Pin_2), J3.4 (Pin_4), J3.6 (Pin_6), J3.8 (Pin_8), J4.2 (Pin_2), J4.4 (Pin_4), J4.6 (Pin_6), J4.8 (Pin_8), H1.1, H2.1, H3.1, H4.1
- net NEUT: now also PS1.1 (AC/N), J6.1 (Pin_1)
- no-connect marks 36 -> 28
Other:
- moved on the sheet: J5
Changed lines of the file:
@@
 Sheet 1 1
 Title "Plug-Pass 120V RFID Control Module"
-Date "2020-05-28"
-Rev "v1.2"
+Date "2020-06-18"
+Rev "v2.0"
 Comp "Clatskanie People's Utility District"
 Comment1 "designed by: Paul Dockery, Power Manager"
@@
 F 0 "J1" H 8350 2250 50  0000 C CNN
 F 1 "Conn_01x06" V 8400 1900 50  0000 C CNN
-F 2 "Plug_Pass:PinSocket_1x06_P2.54mm_Vertical" H 8300 1950 50  0001 C CNN
+F 2 "Plug_Pass:RTC_PinHeader" H 8300 1950 50  0001 C CNN
 F 3 "~" H 8300 1950 50  0001 C CNN
 	1    8300 1950
@@
 F 0 "J2" H 3500 2350 50  0000 L CNN
 F 1 "Conn_01x08" V 3600 1650 50  0000 L CNN
-F 2 "Plug_Pass:PinSocket_1x08_P2.54mm_Vertical" H 3500 1950 50  0001 C CNN
+F 2 "Plug_Pass:PN532_NFC_PinSocket" H 3500 1950 50  0001 C CNN
 F 3 "~" H 3500 1950 50  0001 C CNN
 	1    3500 1950
@@
 	4700 4400 4600 4400
 $Comp
-L Plug_Pass:Conn_WallSocket_Earth J5
-U 1 1 5EAEB62E
-P 6750 4850
-F 0 "J5" H 7004 4861 50  0000 L CNN
-F 1 "Conn_WallSocket_Earth" V 7150 4550 50  0000 L CNN
-F 2 "" H 6450 4950 50  0001 C CNN
-F 3 "~" H 6450 4950 50  0001 C CNN
-	1    6750 4850
-	1    0    0    -1
-$EndComp
-$Comp
 L power:+3V3 #PWR03
 U 1 1 5E9D4087
@@
 $EndComp
 Wire Wire Line
-	5850 4650 6550 4650
+	5850 4650 6500 4650
 Text Label 3100 6400 0    50   ~ 0
 VCC
@@
 Text Notes 3250 2400 1    50   ~ 0
 Female socket connector \nfor PN532 NFC Module
-Text Notes 3050 3300 1    50   ~ 0
+Text Notes 2850 3250 1    50   ~ 0
 Ribbon connector for\npower supply and\nrelay shield
 $Comp
@@
 P 6050 2050
 F 0 "A1" H 5600 3000 50  0000 C CNN
-F 1 "Arduino_Nano_v3.x" H 6600 1050 50  0000 C CNN
-F 2 "Plug_Pass:Arduino_Nano_WithMountingHoles" H 6050 2050 50  0001 C CIN
+F 1 "Arduino_Nano_Every" H 6600 1050 50  0000 C CNN
+F 2 "Plug_Pass:NANO_33_Footprint_SMD_Castell" H 6050 2050 50  0001 C CIN
 F 3 "http://www.mouser.com/pdfdocs/Gravitech_Arduino_Nano3_0.pdf" H 6050 2050 50  0001 C CNN
 	1    6050 2050
@@
 	5650 5350 5550 5350
 $Comp
-L Plug_Pass:TDPT-1017503 J10
-U 1 1 5E984D8C
-P 5550 7050
-F 0 "J10" V 5400 7050 50  0000 L CNN
-F 1 "TDPT-1017503" H 4900 6950 50  0000 L CNN
-F 2 "Plug_Pass:TDPT_2P_6.35MM" H 5750 7250 60  0001 L CNN
-F 3 "https://media.digikey.com/pdf/Data%20Sheets/Phoenix%20Contact%20PDFs/1017503_Ds.pdf" H 5750 7350 60  0001 L CNN
-F 4 "277-17514-ND" H 5750 7450 60  0001 L CNN "Digi-Key_PN"
-F 5 "1017503" H 5750 7550 60  0001 L CNN "MPN"
-F 6 "Connectors, Interconnects" H 5750 7650 60  0001 L CNN "Category"
-F 7 "Terminal Blocks - Wire to Board" H 5750 7750 60  0001 L CNN "Family"
-F 8 "https://media.digikey.com/pdf/Data%20Sheets/Phoenix%20Contact%20PDFs/1017503_Ds.pdf" H 5750 7850 60  0001 L CNN "DK_Datasheet_Link"
-F 9 "https://www.digikey.com/product-detail/en/phoenix-contact/1017503/277-17514-ND/9346604" H 5750 7950 60  0001 L CNN "DK_Detail_Page"
-F 10 "TERM BLK 2P SIDE ENT 5.08MM PCB" H 5750 8050 60  0001 L CNN "Description"
-F 11 "On Shore Technology Inc." H 5750 8150 60  0001 L CNN "Manufacturer"
-F 12 "Active" H 5750 8250 60  0001 L CNN "Status"
-	1    5550 7050
-	0    -1   1    0
-$EndComp
-$Comp
-L power:Earth #PWR04
-U 1 1 5E9EA062
-P 5850 7150
-F 0 "#PWR04" H 5850 6900 50  0001 C CNN
-F 1 "Earth" H 5850 7000 50  0001 C CNN
-F 2 "" H 5850 7150 50  0001 C CNN
-F 3 "~" H 5850 7150 50  0001 C CNN
-	1    5850 7150
-	0    1    -1   0
-$EndComp
-$Comp
 L Plug_Pass:Conn_02x04_Odd_Even J3
 U 1 1 5E9F6D64
 P 3550 2750
 F 0 "J3" H 3600 2950 50  0000 C CNN
-F 1 "Conn_02x04_Odd_Even" V 3950 2600 50  0000 C CNN
-F 2 "Plug_Pass:IDC-Header_2x04_P2.54mm_Vertical" H 3550 2750 50  0001 C CNN
+F 1 "Conn_02x04_Odd_Even" V 4100 2600 50  0000 C CNN
+F 2 "Plug_Pass:IDC-Header_2x04_P2.54mm_Vertical_Small" H 3550 2750 50  0001 C CNN
 F 3 "~" H 3550 2750 50  0001 C CNN
 	1    3550 2750
 	-1   0    0    -1
 $EndComp
-NoConn ~ 3250 2650
-NoConn ~ 3250 2750
-NoConn ~ 3250 2850
-NoConn ~ 3250 2950
 Text Notes 2200 6750 1    50   ~ 0
 Ribbon connector for\npower supply and\nrelay shield
@@
 P 2900 6300
 F 0 "J4" H 2950 6500 50  0000 C CNN
-F 1 "Conn_02x04_Odd_Even" V 3300 6150 50  0000 C CNN
+F 1 "Conn_02x04_Odd_Even" V 3450 6150 50  0000 C CNN
 F 2 "Plug_Pass:IDC-Header_2x04_P2.54mm_Vertical" H 2900 6300 50  0001 C CNN
 F 3 "~" H 2900 6300 50  0001 C CNN
@@
 	-1   0    0    -1
 $EndComp
-NoConn ~ 2600 6200
-NoConn ~ 2600 6300
-NoConn ~ 2600 6400
-NoConn ~ 2600 6500
 $Comp
 L Plug_Pass:G5V-1-DC5 RLY2
@@
 	5450 7050 4950 7050
 Wire Wire Line
-	5450 7150 5450 7300
-Wire Wire Line
 	4050 7050 4150 7050
 Wire Wire Line
@@
 NoConn ~ 4800 5600
 NoConn ~ 4800 4600
-$Comp
-L Plug_Pass:GNDREF #PWR0108
-U 1 1 5ED94C7D
-P 5450 7300
-F 0 "#PWR0108" H 5450 7050 50  0001 C CNN
-F 1 "GNDREF" H 5450 7150 50  0000 C CNN
-F 2 "" H 5450 7300 50  0001 C CNN
-F 3 "" H 5450 7300 50  0001 C CNN
-	1    5450 7300
-	-1   0    0    -1
-$EndComp
 Wire Notes Line
 	6150 5300 6150 7350
@@
 	5750 7350 5750 5600
 Wire Notes Line
-	5750 5600 5200 5600
-Wire Notes Line
-	5200 5600 5200 4500
-Wire Notes Line
-	5200 4500 4850 4500
+	5350 5600 5350 4500
 Wire Notes Line
 	4850 4500 4850 4250
@@
 	4850 4250 7400 4250
 Wire Wire Line
-	6100 5050 6550 5050
-Wire Wire Line
-	6100 5050 6100 7150
-Wire Wire Line
-	6100 7150 5850 7150
-Wire Wire Line
 	5950 4850 5950 7050
 Wire Wire Line
 	5950 7050 5850 7050
 Wire Wire Line
-	5950 4850 6550 4850
+	5950 4850 6500 4850
 Text Label 4600 5600 1    50   ~ 0
 RLY1-Pin
@@
 Wire Notes Line
 	3200 750  3200 500
+$Comp
+L Plug_Pass:Conn_WallSocket_Earth J5
+U 1 1 5EAEB62E
+P 6700 4850
+F 0 "J5" H 6954 4861 50  0000 L CNN
+F 1 "Conn_WallSocket_Earth" V 7100 4550 50  0000 L CNN
+F 2 "" H 6400 4950 50  0001 C CNN
+F 3 "~" H 6400 4950 50  0001 C CNN
+	1    6700 4850
+	1    0    0    -1
+$EndComp
+Connection ~ 6500 4650
+Wire Wire Line
+	6500 4650 6550 4650
+Connection ~ 6500 4850
+Wire Wire Line
+	6500 4850 6550 4850
+$Comp
+L Plug_Pass:GNDREF #PWR0108
+U 1 1 5EED00AE
+P 6350 5050
+F 0 "#PWR0108" H 6350 4800 50  0001 C CNN
+F 1 "GNDREF" H 6350 4900 50  0000 C CNN
+F 2 "" H 6350 5050 50  0001 C CNN
+F 3 "" H 6350 5050 50  0001 C CNN
+	1    6350 5050
+	-1   0    0    -1
+$EndComp
+Wire Wire Line
+	6500 5050 6350 5050
+$Comp
+L Plug_Pass:Screw_Terminal_01x01 J6
+U 1 1 5EED20BF
+P 5650 7050
+F 0 "J6" H 5730 7092 50  0000 L CNN
+F 1 "Screw_Terminal_01x01" H 5350 6950 50  0000 L CNN
+F 2 "Plug_Pass:PLH5-1_75" H 5650 7050 50  0001 C CNN
+F 3 "~" H 5650 7050 50  0001 C CNN
+	1    5650 7050
+	1    0    0    -1
+$EndComp
+$Comp
+L Plug_Pass:MountingHole_Pad H4
+U 1 1 5EEA4DE0
+P 2850 5600
+F 0 "H4" V 2804 5750 50  0000 L CNN
+F 1 "MountingHole_Pad" V 2895 5750 50  0000 L CNN
+F 2 "Plug_Pass:Ground_Pad" H 2850 5600 50  0001 C CNN
+F 3 "~" H 2850 5600 50  0001 C CNN
+	1    2850 5600
+	0    -1   -1   0
+$EndComp
+$Comp
+L Plug_Pass:MountingHole_Pad H3
+U 1 1 5EEA5BFE
+P 2850 5400
+F 0 "H3" V 2804 5550 50  0000 L CNN
+F 1 "MountingHole_Pad" V 2895 5550 50  0000 L CNN
+F 2 "Plug_Pass:Ground_Pad" H 2850 5400 50  0001 C CNN
+F 3 "~" H 2850 5400 50  0001 C CNN
+	1    2850 5400
+	0    -1   -1   0
+$EndComp
+$Comp
+L Plug_Pass:MountingHole_Pad H2
+U 1 1 5EEA5DC0
+P 2850 5200
+F 0 "H2" V 2804 5350 50  0000 L CNN
+F 1 "MountingHole_Pad" V 2895 5350 50  0000 L CNN
+F 2 "Plug_Pass:Ground_Pad" H 2850 5200 50  0001 C CNN
+F 3 "~" H 2850 5200 50  0001 C CNN
+	1    2850 5200
+	0    -1   -1   0
+$EndComp
+$Comp
+L Plug_Pass:MountingHole_Pad H1
+U 1 1 5EEA5F35
+P 2850 5000
+F 0 "H1" V 2804 5150 50  0000 L CNN
+F 1 "MountingHole_Pad" V 2895 5150 50  0000 L CNN
+F 2 "Plug_Pass:Ground_Pad" H 2850 5000 50  0001 C CNN
+F 3 "~" H 2850 5000 50  0001 C CNN
+	1    2850 5000
+	0    -1   -1   0
+$EndComp
+$Comp
+L Plug_Pass:GNDREF #PWR0109
+U 1 1 5EEAA57F
+P 3150 5300
+F 0 "#PWR0109" H 3150 5050 50  0001 C CNN
+F 1 "GNDREF" H 3155 5127 50  0000 C CNN
+F 2 "" H 3150 5300 50  0001 C CNN
+F 3 "" H 3150 5300 50  0001 C CNN
+	1    3150 5300
+	-1   0    0    -1
+$EndComp
+Wire Wire Line
+	2950 5000 2950 5200
+Wire Wire Line
+	2950 5200 2950 5300
+Connection ~ 2950 5200
+Wire Wire Line
+	2950 5400 2950 5600
+Connection ~ 2950 5400
+Wire Wire Line
+	2950 5300 3150 5300
+Connection ~ 2950 5300
+Wire Wire Line
+	2950 5300 2950 5400
+$Comp
+L Plug_Pass:GNDREF #PWR0110
+U 1 1 5EEB5119
+P 3250 3050
+F 0 "#PWR0110" H 3250 2800 50  0001 C CNN
+F 1 "GNDREF" H 3255 2877 50  0000 C CNN
+F 2 "" H 3250 3050 50  0001 C CNN
+F 3 "" H 3250 3050 50  0001 C CNN
+	1    3250 3050
+	-1   0    0    -1
+$EndComp
+Wire Wire Line
+	3250 2650 3250 2750
+Wire Wire Line
+	3250 2750 3250 2850
+Connection ~ 3250 2750
+Wire Wire Line
+	3250 2850 3250 2950
+Connection ~ 3250 2850
+Wire Wire Line
+	3250 2950 3250 3050
+Connection ~ 3250 2950
+$Comp
+L Plug_Pass:GNDREF #PWR0111
+U 1 1 5EEBE750
+P 2600 6600
+F 0 "#PWR0111" H 2600 6350 50  0001 C CNN
+F 1 "GNDREF" H 2600 6450 50  0000 C CNN
+F 2 "" H 2600 6600 50  0001 C CNN
+F 3 "" H 2600 6600 50  0001 C CNN
+	1    2600 6600
+	-1   0    0    -1
+$EndComp
+Wire Wire Line
+	2600 6200 2600 6300
+Wire Wire Line
+	2600 6300 2600 6400
+Connection ~ 2600 6300
+Wire Wire Line
+	2600 6400 2600 6500
+Connection ~ 2600 6400
+Wire Wire Line
+	2600 6500 2600 6600
+Connection ~ 2600 6500
+Text Label 5450 7050 2    50   ~ 0
+NEUT
+Text Label 4950 7050 0    50   ~ 0
+NEUT
+Wire Notes Line
+	4850 4500 5350 4500
+Wire Notes Line
+	5350 5600 5750 5600
 $EndSCHEMATC
