File: hardware/PCB/Plug_Pass.sch (KiCad schematic (older format))
At the start: 16 parts, among them J1 Conn_01x06, J2 Conn_01x08, J3 Conn_02x04_Odd_Even, J4 Conn_02x04_Odd_Even, J5 Conn_WallSocket_Earth, J6 Screw_Terminal_01x01, J8 QuickDisconnect, J9 QuickDisconnect

Commit message: Add files via upload
Parts:
- removed J3: Conn_02x04_Odd_Even, Plug_Pass:IDC-Header_2x04_P2.54mm_Vertical_Small, symbol Plug_Pass:Conn_02x04_Odd_Even
- removed J4: Conn_02x04_Odd_Even, Plug_Pass:IDC-Header_2x04_P2.54mm_Vertical, symbol Plug_Pass:Conn_02x04_Odd_Even
Connections:
- net labels added: AC-L
- wire segments 78 -> 76
- no-connect marks 28 -> 23
Other:
- note removed: "AC Shield\nfor Power Supply and Relay shield"
- note removed: "Arduino Shield\nfor Arduino Nano, PN532, and RTC3231 sockets"
- note removed: "Ribbon connector for\npower supply and\nrelay shield"
- moved on the sheet: J2

Commit message: Add files via upload
Parts:
- removed A1: Arduino_Nano_Every, Plug_Pass:NANO_33_Footprint_SMD_Castell, symbol Plug_Pass:Arduino_Nano_v3.x
- removed H1, H2, H3, H4: MountingHole_Pad, Plug_Pass:Ground_Pad, symbol Plug_Pass:MountingHole_Pad
- removed J1: Conn_01x06, Plug_Pass:RTC_PinHeader, symbol Plug_Pass:Conn_01x06
- removed J2: Conn_01x08, Plug_Pass:PN532_NFC_PinSocket, symbol Plug_Pass:Conn_01x08
- removed J5: Conn_WallSocket_Earth, symbol Plug_Pass:Conn_WallSocket_Earth
- removed J6: Screw_Terminal_01x01, Plug_Pass:PLH5-1_75, symbol Plug_Pass:Screw_Terminal_01x01
- removed J8, J9: QuickDisconnect, symbol Plug_Pass:QuickDisconnect
- removed PS1: IRM-05-5, Plug_Pass:Converter_ACDC_MeanWell_IRM-05-xx_THT, symbol Plug_Pass:IRM-05-5
- added B1: CR1220, Plug_Pass:CR1220, symbol Plug_Pass:BATTERYCR1220_SMT
- added C1, C17, C18, C2, C20, C3, C8: 0.1µF, Plug_Pass:0603-1608X90N, symbol Plug_Pass:C_Small
- added C10, C13: 100pF, Plug_Pass:0603-1608X90N, symbol Plug_Pass:C_Small
- added C11, C14: 220pF, Plug_Pass:0402-1005X55N, symbol Plug_Pass:C_Small
- added C12, C16, C7, C9: NC, Plug_Pass:0805-R2013X50N, symbol Plug_Pass:C_Small
- added C15, C6: 22pF, Plug_Pass:0402-1005X55N, symbol Plug_Pass:C_Small
- added C19, C21, C22, C4, C5: 10µF, Plug_Pass:0603-1608X90N, symbol Plug_Pass:C_Small
- added C23: 1000pF, Plug_Pass:0603-1608X90N, symbol Plug_Pass:C_Small
- added C24, C25: 33pF, Plug_Pass:0603-1608X90N, symbol Plug_Pass:C_Small
- added C26, C28: 1µF, Plug_Pass:0402-1005X55N, symbol Plug_Pass:C_Small
- added C27, C31: 4,7uF_16V, Plug_Pass:CAPAE430X550N, symbol Plug_Pass-rescue:CP_Small-Plug_Pass
- added C29, C30, C33: 100nF, Plug_Pass:0402-1005X55N, symbol Plug_Pass:C_Small
- added C32: 1uF, Plug_Pass:0402-1005X55N, symbol Plug_Pass:C_Small
- added D1: 0025_SS1P3L-M3_84A, Plug_Pass:DO220AAL, symbol Plug_Pass:0025_SS1P3L-M3_84A
- added F1: MFFSMF050, Plug_Pass:0603-1608X90N, symbol Plug_Pass:Thermistor
- added GND1, GND2, GND3, GND4, GND5: GND, Plug_Pass:Ground_Pad, symbol Plug_Pass:MountingHole_Pad
- added IC1: DS3231M, Package_SO:SOIC-16W_7.5x10.3mm_P1.27mm, symbol Plug_Pass:DS3231M
- added IC2: PN532, Plug_Pass:HVQFN40-6X6, symbol Plug_Pass:PN532
- added IC3: VREG_SOT23-5, Plug_Pass:SOT23-5, symbol Plug_Pass:VREG_SOT23-5
- added IC4: FT232RL, digikey-footprints:SSOP-28_W5.30mm, symbol Plug_Pass:FT232RL-REEL
- added IC5: ATMEGA328P-AUR, digikey-footprints:TQFP-32_7x7mm, symbol Plug_Pass:ATMEGA328P-AUR
- added J1: USB_B_Micro, Plug_Pass:MOLEX_1051330001, symbol Plug_Pass:USB_B_Micro
- added J2: 505568-0271, Plug_Pass:5055680271, symbol Plug_Pass:505568-0271
- added L1: Yellow, Plug_Pass:LEDC1608X80N-AK, symbol Plug_Pass:LED_Small
- added L2, L5: FERRITE, Plug_Pass:0805-R2013X50N, symbol Plug_Pass:Ferrite_Bead_Small
- added L3, L4: 560nH, Plug_Pass:0805-R2013X50N, symbol Plug_Pass:L_Small
- added NEUT1: NEUT, Plug_Pass:Ground_Pad, symbol Plug_Pass:MountingHole_Pad
- added PS1: IRM-03-5, Converter_ACDC:Converter_ACDC_MeanWell_IRM-03-xx_SMD, symbol Plug_Pass:IRM-03-5
- added PWR1, TX1: Green, Plug_Pass:LEDC1608X80N-AK, symbol Plug_Pass:LED_Small
- added R1, R6: 1.5, Plug_Pass:0402-1005X55N, symbol Plug_Pass:R_Small
- added R10, R11, R12, R9: 330, Plug_Pass:0402-1005X55N, symbol Plug_Pass:R_Small
- added R2, R4: 10k, Plug_Pass:0402-1005X55N, symbol Device:R_Small
- added R3, R5: NC, Plug_Pass:R0201, symbol Plug_Pass:R_Small
- added R7: 1.0k, Plug_Pass:0402-1005X55N, symbol Plug_Pass:R_Small
- added R8: 1.69k, Plug_Pass:0402-1005X55N, symbol Plug_Pass:R_Small
- added RP1: 1k, Plug_Pass:CAY16, symbol Plug_Pass:0005_064R_1K___CAY16-102J4LF
- added RX1: Red, Plug_Pass:LEDC1608X80N-AK, symbol Plug_Pass:LED_Small
- added SW1: RESET, Plug_Pass:C&K_PTS820_NO_HOLES, symbol Plug_Pass:SW_Push
- added TP1: TX1_POST, Plug_Pass:TESTPOINT_ROUND_1MM, symbol Plug_Pass:TESTPOINT
- added TP2, TP5: TGND, Plug_Pass:TESTPOINT_ROUND_1MM, symbol Plug_Pass:TESTPOINT
- added TP3: TX2_POST, Plug_Pass:TESTPOINT_ROUND_1MM, symbol Plug_Pass:TESTPOINT
- added TP4: TX1_PRE, Plug_Pass:TESTPOINT_ROUND_1MM, symbol Plug_Pass:TESTPOINT
- added TP6: TX2_PRE, Plug_Pass:TESTPOINT_ROUND_1MM, symbol Plug_Pass:TESTPOINT
- added TP7: RX, Plug_Pass:TESTPOINT_ROUND_1MM, symbol Plug_Pass:TESTPOINT
- added TP8: D11, Plug_Pass:TESTPOINT_ROUND_1MM, symbol Plug_Pass:TESTPOINT
- added TP9: D+1, Plug_Pass:TESTPOINT_ROUND_1MM, symbol Plug_Pass:TESTPOINT
- added Y1: 27.12MHz, Plug_Pass:7M27120MAAJT, symbol Plug_Pass:Crystal_GND24_Small
- added Y2: 16MHz, Plug_Pass:CSTNE16M0V51Z000R0, symbol Plug_Pass:0011_CSTCE16M0V53-R0
- RLY1: footprint Plug_Pass:RLY-T9AS5D22-5 -> Plug_Pass:RLY-T9AS1D22-5; symbol Plug_Pass:G5LE-14_DC5 -> Plug_Pass:T9AS1D22-5
Connections:
- net labels added: +3.3V, AVDD, BAT+, BAT-, D+, D-, DGND, LDO, MISO(D12), MOSI(D11), PVDD, RESET, RLY1, RLY2, RLY2-Pin(D2), RX, RX_RED, SCK(D13), SCL(A5), SDA(A4), SS(D10), TGND1, TGND2, TVDD, TX, TX1, TX2, TX_GREEN, VUSB
- net labels removed: IRQ, RLY1-Pin, RSTO, VAC
- wire segments 76 -> 356
- no-connect marks 23 -> 46
Other:
- note removed: "Female socket connector \nfor PN532 NFC Module"
- note removed: "Female socket connector \nfor RTC3231 module"
- note removed: "Primary voltages to relay and outlets are hand\nwired, not printed on circuit board."
- moved on the sheet: RLY2

Commit message: Add files via upload
Parts:
- added J3: Conn_02x03, Plug_Pass:PinHeader_2x03_P1.00mm_Vertical_SMD, symbol Plug_Pass:Conn_01x06
- added S1: 218-4LPST, Plug_Pass:SOIC127P844X265-8N, symbol Plug_Pass:218-4LPST
Connections:
- net +5V: now also RP1.6 (2), J3.4 (Pin_4); no longer RP1.7 (2)
- net GNDREF: now also J3.2 (Pin_2)
- net MISO: now also J3.3 (Pin_3), S1.7; no longer IC2.29 (MISO)
- net MOSI: now also J3.1 (Pin_1), S1.8; no longer IC2.28 (MOSI/SDA/HSU_TX)
- net RESET: now also J3.6 (Pin_6), S1.5; no longer C30.1, RP1.2 (1), SW1.2
- net RX: now also RP1.7 (2); no longer RP1.3 (1)
- net SCK: now also J3.5 (Pin_5), S1.6; no longer IC2.30 (SCK), R12.1
- net TX: now also RP1.5 (2); no longer RP1.4 (1)
- net RX1: now reaches C23.2, IC2.10 (RX), R7.1
- net VMID: now reaches C20.2, IC2.9 (VMID), R7.2
- net at IC5.30 (PD0): now also RP1.2 (1); no longer RP1.6 (2)
- net at IC5.31 (PD1): now also RP1.4 (1); no longer RP1.5 (2)
- new net MISO-1: IC2.29 (MISO), S1.2
- new net MOSI-1: IC2.28 (MOSI/SDA/HSU_TX), S1.1
- new net RESET-1: C30.1, RP1.3 (1), S1.4, SW1.2
- new net SCK-1: IC2.30 (SCK), R12.1, S1.3
Other:
- moved on the sheet: GND2, GND3, GND4, GND5, SW1, Y2

Commit message: Board update v3.2
Parts:
- removed C12, C16, C7, C9: NC, Plug_Pass:0805-R2013X50N, symbol Plug_Pass:C_Small
- removed IC3: VREG_SOT23-5, Plug_Pass:SOT23-5, symbol Plug_Pass:VREG_SOT23-5
- removed J3: Conn_02x03, Plug_Pass:PinHeader_2x03_P1.00mm_Vertical_SMD, symbol Plug_Pass:Conn_01x06
- removed R3, R5: NC, Plug_Pass:R0201, symbol Plug_Pass:R_Small
- removed TP1: TX1_POST, Plug_Pass:TESTPOINT_ROUND_1MM, symbol Plug_Pass:TESTPOINT
- removed TP2, TP5: TGND, Plug_Pass:TESTPOINT_ROUND_1MM, symbol Plug_Pass:TESTPOINT
- removed TP3: TX2_POST, Plug_Pass:TESTPOINT_ROUND_1MM, symbol Plug_Pass:TESTPOINT
- removed TP4: TX1_PRE, Plug_Pass:TESTPOINT_ROUND_1MM, symbol Plug_Pass:TESTPOINT
- removed TP6: TX2_PRE, Plug_Pass:TESTPOINT_ROUND_1MM, symbol Plug_Pass:TESTPOINT
- removed TP7: RX, Plug_Pass:TESTPOINT_ROUND_1MM, symbol Plug_Pass:TESTPOINT
- removed Y2: 16MHz, Plug_Pass:CSTNE16M0V51Z000R0, symbol Plug_Pass:0011_CSTCE16M0V53-R0
- added C35, C36: 22pF, Plug_Pass:0603-1608X90N, symbol Plug_Pass:C_Small
- added CR1: LD1117V33, footprints:LD1117V33, symbol 2021-06-09_00-46-52:LD1117V33
- added D2: 1N4148WS, SODFL2512X100N, symbol 1N4148WS:1N4148WS
- added J3: Conn_01x08, Connector_PinSocket_2.54mm:PinSocket_1x08_P2.54mm_Vertical_SMD_Pin1Right, symbol Plug_Pass:Conn_01x08
- added J4: Conn_01x02, Connector_PinHeader_2.54mm:PinHeader_1x02_P2.54mm_Vertical, symbol Connector_Generic:Conn_01x02
- added Q1: 2N3904, TO92127P495H495-3, symbol 2N3904:2N3904
- added R13: 4.7k, Plug_Pass:0402-1005X55N, symbol Plug_Pass:R_Small
- added Y2: ECS-51-20-4, ECS-51-20-4:XTAL_ECS-51-20-4, symbol ECS-51-20-4:ECS-51-20-4
- C10, C13: value 100pF -> 62pF; footprint Plug_Pass:0603-1608X90N -> Capacitor_SMD:C_0805_2012Metric
- C15, C6: value 22pF -> 14pF; footprint Plug_Pass:0402-1005X55N -> Capacitor_SMD:C_0805_2012Metric
- R1, R6: value 1.5 -> 2; footprint Plug_Pass:0402-1005X55N -> Resistor_SMD:R_0805_2012Metric
- R8: footprint Plug_Pass:0402-1005X55N -> Resistor_SMD:R_0805_2012Metric
Connections:
- net +3V3: now also IC2.17 (I1), IC2.38 (RSTPD_N), CR1.2 (VOUT); no longer IC2.16 (I0)
- net +5V: now also RLY1.5 (COIL), RLY2.2 (COIL), CR1.3 (VIN), D2.C, J3.4 (Pin_4); no longer RLY2.5 (COM), RLY2.6 (COM)
- net GNDREF: now also IC2.16 (I0), RLY2.10 (NO), C35.1, C36.1, CR1.1 (ADJ/GND), J3.2 (Pin_2), J3.3 (Pin_3), Q1.1; no longer IC2.17 (I1), RLY1.2 (COIL), RLY2.9 (COIL)
- net MISO: now also J3.7 (Pin_7)
- net MOSI: now also J3.6 (Pin_6)
- net RESET: now also C30.1, RP1.3 (1), SW1.2, J3.1 (Pin_1); no longer S1.5
- net SCK: now also R12.1, J3.8 (Pin_8)
- net SCK-1: no longer R12.1
- net SS: now also S1.5, J3.5 (Pin_5); no longer IC2.27 (NSS/P50_SCL/HSU_RX)
- net at IC5.7 (PB6): now also C36.2, Y2.2
- net at IC5.8 (PB7): now also C35.2, Y2.1
- removed net RESET-1: C30.1, RP1.3 (1), S1.4, SW1.2
- removed net RLY1: RLY1.5 (COIL), RLY2.10 (NO)
- net RLY2 renamed RLY
- net RLY: now also J4.2 (Pin_2), R13.2; no longer RLY2.2 (COIL)
- new net: D2.A, RLY1.2 (COIL), RLY2.5 (COM), RLY2.6 (COM)
- new net: Q1.3, RLY2.9 (COIL)
- new net: J4.1 (Pin_1), Q1.2, R13.1
- new net SS-1: IC2.27 (NSS/P50_SCL/HSU_RX), S1.4
Other:
- moved on the sheet: C21, C22, RLY1, RLY2

Commit message: Update 4
Parts:
- removed C1, C17, C18, C2, C20, C3, C8: 0.1µF, Plug_Pass:0603-1608X90N, symbol Plug_Pass:C_Small
- removed C10, C13: 62pF, Capacitor_SMD:C_0805_2012Metric, symbol Plug_Pass:C_Small
- removed C11, C14: 220pF, Plug_Pass:0402-1005X55N, symbol Plug_Pass:C_Small
- removed C15, C6: 14pF, Capacitor_SMD:C_0805_2012Metric, symbol Plug_Pass:C_Small
- removed C19, C22, C4, C5: 10µF, Plug_Pass:0603-1608X90N, symbol Plug_Pass:C_Small
- removed C23: 1000pF, Plug_Pass:0603-1608X90N, symbol Plug_Pass:C_Small
- removed C24, C25: 33pF, Plug_Pass:0603-1608X90N, symbol Plug_Pass:C_Small
- removed CR1: LD1117V33, footprints:LD1117V33, symbol 2021-06-09_00-46-52:LD1117V33
- removed IC2: PN532, Plug_Pass:HVQFN40-6X6, symbol Plug_Pass:PN532
- removed J2: 505568-0271, Plug_Pass:5055680271, symbol Plug_Pass:505568-0271
- removed J4: Conn_01x02, Connector_PinHeader_2.54mm:PinHeader_1x02_P2.54mm_Vertical, symbol Connector_Generic:Conn_01x02
- removed L1: Yellow, Plug_Pass:LEDC1608X80N-AK, symbol Plug_Pass:LED_Small
- removed L2, L5: FERRITE, Plug_Pass:0805-R2013X50N, symbol Plug_Pass:Ferrite_Bead_Small
- removed L3, L4: 560nH, Plug_Pass:0805-R2013X50N, symbol Plug_Pass:L_Small
- removed R1, R6: 2, Resistor_SMD:R_0805_2012Metric, symbol Plug_Pass:R_Small
- removed R12: 330, Plug_Pass:0402-1005X55N, symbol Plug_Pass:R_Small
- removed RP1: 1k, Plug_Pass:CAY16, symbol Plug_Pass:0005_064R_1K___CAY16-102J4LF
- removed S1: 218-4LPST, Plug_Pass:SOIC127P844X265-8N, symbol Plug_Pass:218-4LPST
- removed TP8: D11, Plug_Pass:TESTPOINT_ROUND_1MM, symbol Plug_Pass:TESTPOINT
- removed TP9: D+1, Plug_Pass:TESTPOINT_ROUND_1MM, symbol Plug_Pass:TESTPOINT
- removed Y1: 27.12MHz, Plug_Pass:7M27120MAAJT, symbol Plug_Pass:Crystal_GND24_Small
- added GND6: GND, Plug_Pass:Ground_Pad, symbol Plug_Pass:MountingHole_Pad
- added R9: 1k, Plug_Pass:0402-1005X55N, symbol Plug_Pass:R_Small
- added U1: TC1108-3.3VDBTR, SOT230P700X180-4N, symbol SamacSys_Parts:TC1108-3.3VDBTR
- C10: renamed from C21; value 10µF -> 1µF
- C6: renamed from C27; value 4,7uF_16V -> 4.7uF
- C7: renamed from C31; value 4,7uF_16V -> 4.7uF
- IC2: renamed from IC4; footprint digikey-footprints:SSOP-28_W5.30mm -> Plug_Pass:SSOP-28_W5.30mm
- IC3: renamed from IC5; footprint digikey-footprints:TQFP-32_7x7mm -> Plug_Pass:TQFP-32_7x7mm
- R7: value 1.0k -> 1k; Description Thick Film Resistors - SMD 1K ohm 5% 50V General Purpose -> Thick Film Resistors - SMD 4.7k OHM 1%; MPN RC0402JR-131KL -> RC0402FR-074K7L
- R8: value 1.69k -> 1k; footprint Resistor_SMD:R_0805_2012Metric -> Plug_Pass:0402-1005X55N; Description Thick Film Resistors - SMD 1.69K OHM 1% -> Thick Film Resistors - SMD 4.7k OHM 1%; MPN RC0402FR-071K69L -> RC0402FR-074K7L
- renumbered C36 to C1, C32 to C11, C35 to C2, C29 to C3, C26 to C4, C28 to C5, C33 to C8, C30 to C9, J3 to J2, R4 to R1, R10 to R3, R11 to R4, R9 to R5, R13 to R6, Y2 to Y1
Connections:
- net RX1 is gone; now on net RESET: R7.1
- net VMID is gone; now on net +5V: R7.2
- net +3V3: now also C10.1, U1.3 (VOUT)
- net +5V: now also U1.1 (VIN); no longer C10.1
- net GNDREF: now also GND6.1, U1.2 (GND_1), U1.4 (GND_2)
- net RX: now also R8.2
- net TX: now also R9.2
- net at IC3.30 (PD0): now also R8.1
- net at IC3.31 (PD1): now also R9.1
- no-connect marks 46 -> 31
Other:
- moved on the sheet: B1, C1, C10, C11, C2, C3, C4, C5, C6, C7, C8, C9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
